File: rpi-nrf52840-hat/rpi-nrf52840-hat.kicad_pcb (KiCad board)
At the start: 2 copper layers, 65 x 56 mm, 31 parts, among them J1 Conn_02x04_Odd_Even, J2 Raspberry_Pi_4, J3 Conn_02x04_Odd_Even, U1 E73-2G4M08S1C, U2 24C32, X1 32.768kHz 12.5pF

Commit message: remove populate_jlc_library and convert to kifab
Parts:
- D1: footprint rpi-nrf52840-hat:LED_RGB_1.6x1.5mm_CA_P4-1615 -> project:LED_RGB_1.6x1.5mm_CA_P4-1615
- J1, J3: footprint Connector_PinHeader_2.54mm:PinHeader_2x04_P2.54mm_Vertical -> project:PinHeader_2x04_P2.54mm_Vertical
- J2: footprint Connector_PinSocket_2.54mm:PinSocket_2x20_P2.54mm_Vertical -> project:PinSocket_2x20_P2.54mm_Vertical
- MH1, MH2, MH3, MH4: footprint MountingHole:MountingHole_2.7mm_M2.5 -> project:MountingHole_2.7mm_M2.5
- TP1: footprint Connector_PinHeader_2.54mm:PinHeader_1x01_P2.54mm_Vertical -> project:PinHeader_1x01_P2.54mm_Vertical
Changed lines of the file:
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@@
 		)
 		(embedded_fonts no)
-		(model "${KIPRJMOD}/jlcpcb-lib/jlcpcb.3dshapes/R0603.wrl"
+		(model "${KIPRJMOD}/lib/jlcpcb/jlcpcb.3dshapes/R0603.wrl"
 			(offset
 				(xyz 0 0 0)
@@
 		)
 	)
-	(footprint "MountingHole:MountingHole_2.7mm_M2.5"
+	(footprint "project:MountingHole_2.7mm_M2.5"
 		(locked yes)
 		(layer "F.Cu")
@@
 		)
 		(embedded_fonts no)
-		(model "${KIPRJMOD}/jlcpcb-lib/jlcpcb.3dshapes/R0603.wrl"
+		(model "${KIPRJMOD}/lib/jlcpcb/jlcpcb.3dshapes/R0603.wrl"
 			(offset
 				(xyz 0 0 0)
@@
 		)
 		(embedded_fonts no)
-		(model "${KIPRJMOD}/jlcpcb-lib/jlcpcb.3dshapes/R0603.wrl"
+		(model "${KIPRJMOD}/lib/jlcpcb/jlcpcb.3dshapes/R0603.wrl"
 			(offset
 				(xyz 0 0 0)
@@
 		)
 	)
-	(footprint "Connector_PinHeader_2.54mm:PinHeader_2x04_P2.54mm_Vertical"
+	(footprint "project:PinHeader_2x04_P2.54mm_Vertical"
 		(layer "F.Cu")
 		(at 110 72.81 180)
@@
 		)
 		(embedded_fonts no)
-		(model "${KICAD10_3DMODEL_DIR}/Connector_PinHeader_2.54mm.3dshapes/PinHeader_2x04_P2.54mm_Vertical.step"
+		(model "${KIPRJMOD}/lib/project/project.3dshapes/PinHeader_2x04_P2.54mm_Vertical.step"
 			(offset
 				(xyz 0 0 0)
@@
 		)
 		(embedded_fonts no)
-		(model "${KIPRJMOD}/jlcpcb-lib/jlcpcb.3dshapes/R0603.wrl"
+		(model "${KIPRJMOD}/lib/jlcpcb/jlcpcb.3dshapes/R0603.wrl"
 			(offset
 				(xyz 0 0 0)
@@
 		)
 		(embedded_fonts no)
-		(model "${KIPRJMOD}/jlcpcb-lib/jlcpcb.3dshapes/SOP-8_L4.9-W3.9-P1.27-LS6.0-BL-1.wrl"
+		(model "${KIPRJMOD}/lib/jlcpcb/jlcpcb.3dshapes/SOP-8_L4.9-W3.9-P1.27-LS6.0-BL-1.wrl"
 			(offset
 				(xyz 0 0 0)
@@
 		)
 		(embedded_fonts no)
-		(model "${KIPRJMOD}/jlcpcb-lib/jlcpcb.3dshapes/C0805_L2.0-W1.3-H1.3.wrl"
+		(model "${KIPRJMOD}/lib/jlcpcb/jlcpcb.3dshapes/C0805_L2.0-W1.3-H1.3.wrl"
 			(offset
 				(xyz 0 0 0)
@@
 		)
 		(embedded_fonts no)
-		(model "${KIPRJMOD}/jlcpcb-lib/jlcpcb.3dshapes/WIRELM-SMD_L18.0-W13.0-H3.0-E73-2G4M08S1C.wrl"
+		(model "${KIPRJMOD}/lib/jlcpcb/jlcpcb.3dshapes/WIRELM-SMD_L18.0-W13.0-H3.0-E73-2G4M08S1C.wrl"
 			(offset
 				(xyz 0 0 0)
@@
 		)
 	)
-	(footprint "Connector_PinHeader_2.54mm:PinHeader_1x01_P2.54mm_Vertical"
+	(footprint "project:PinHeader_1x01_P2.54mm_Vertical"
 		(layer "F.Cu")
 		(at 147 59.5)
@@
 		)
 		(embedded_fonts no)
-		(model "${KICAD10_3DMODEL_DIR}/Connector_PinHeader_2.54mm.3dshapes/PinHeader_1x01_P2.54mm_Vertical.step"
+		(model "${KIPRJMOD}/lib/project/project.3dshapes/PinHeader_1x01_P2.54mm_Vertical.step"
 			(offset
 				(xyz 0 0 0)
@@
 		)
 		(embedded_fonts no)
-		(model "${KIPRJMOD}/jlcpcb-lib/jlcpcb.3dshapes/R0603.wrl"
+		(model "${KIPRJMOD}/lib/jlcpcb/jlcpcb.3dshapes/R0603.wrl"
 			(offset
 				(xyz 0 0 0)
@@
 		)
 		(embedded_fonts no)
-		(model "${KIPRJMOD}/jlcpcb-lib/jlcpcb.3dshapes/R0603.wrl"
+		(model "${KIPRJMOD}/lib/jlcpcb/jlcpcb.3dshapes/R0603.wrl"
 			(offset
 				(xyz 0 0 0)
@@
 		)
 		(embedded_fonts no)
-		(model "${KIPRJMOD}/jlcpcb-lib/jlcpcb.3dshapes/C0805_L2.0-W1.3-H1.3.wrl"
+		(model "${KIPRJMOD}/lib/jlcpcb/jlcpcb.3dshapes/C0805_L2.0-W1.3-H1.3.wrl"
 			(offset
 				(xyz 0 0 0)
@@
 		)
 		(embedded_fonts no)
-		(model "${KIPRJMOD}/jlcpcb-lib/jlcpcb.3dshapes/R0603.wrl"
+		(model "${KIPRJMOD}/lib/jlcpcb/jlcpcb.3dshapes/R0603.wrl"
 			(offset
 				(xyz 0 0 0)
@@
 		)
 		(embedded_fonts no)
-		(model "${KIPRJMOD}/jlcpcb-lib/jlcpcb.3dshapes/C0603_L1.6-W0.8-H0.8.wrl"
+		(model "${KIPRJMOD}/lib/jlcpcb/jlcpcb.3dshapes/C0603_L1.6-W0.8-H0.8.wrl"
 			(offset
 				(xyz 0 0 0)
@@
 		)
 		(embedded_fonts no)
-		(model "${KIPRJMOD}/jlcpcb-lib/jlcpcb.3dshapes/R0603.wrl"
+		(model "${KIPRJMOD}/lib/jlcpcb/jlcpcb.3dshapes/R0603.wrl"
 			(offset
 				(xyz 0 0 0)
@@
 		)
 	)
-	(footprint "Connector_PinHeader_2.54mm:PinHeader_2x04_P2.54mm_Vertical"
+	(footprint "project:PinHeader_2x04_P2.54mm_Vertical"
 		(layer "F.Cu")
 		(at 118.5 56.54 90)
@@
 		)
 		(embedded_fonts no)
-		(model "${KICAD10_3DMODEL_DIR}/Connector_PinHeader_2.54mm.3dshapes/PinHeader_2x04_P2.54mm_Vertical.step"
+		(model "${KIPRJMOD}/lib/project/project.3dshapes/PinHeader_2x04_P2.54mm_Vertical.step"
 			(offset
 				(xyz 0 0 0)
@@
 		)
 	)
-	(footprint "MountingHole:MountingHole_2.7mm_M2.5"
+	(footprint "project:MountingHole_2.7mm_M2.5"
 		(locked yes)
 		(layer "F.Cu")
@@
 		(embedded_fonts no)
 	)
-	(footprint "MountingHole:MountingHole_2.7mm_M2.5"
+	(footprint "project:MountingHole_2.7mm_M2.5"
 		(locked yes)
 		(layer "F.Cu")
@@
 		(embedded_fonts no)
 	)
-	(footprint "rpi-nrf52840-hat:LED_RGB_1.6x1.5mm_CA_P4-1615"
+	(footprint "project:LED_RGB_1.6x1.5mm_CA_P4-1615"
 		(layer "F.Cu")
 		(at 132.5 69 -90)
@@
 		)
 		(embedded_fonts no)
-		(model "${KIPRJMOD}/jlcpcb-lib/jlcpcb.3dshapes/R0603.wrl"
+		(model "${KIPRJMOD}/lib/jlcpcb/jlcpcb.3dshapes/R0603.wrl"
 			(offset
 				(xyz 0 0 0)
@@
 		)
 		(embedded_fonts no)
-		(model "${KIPRJMOD}/jlcpcb-lib/jlcpcb.3dshapes/R0603.wrl"
+		(model "${KIPRJMOD}/lib/jlcpcb/jlcpcb.3dshapes/R0603.wrl"
 			(offset
 				(xyz 0 0 0)
@@
 		)
 		(embedded_fonts no)
-		(model "${KIPRJMOD}/jlcpcb-lib/jlcpcb.3dshapes/CRYSTAL-SMD_L3.2-W1.5-1.wrl"
+		(model "${KIPRJMOD}/lib/jlcpcb/jlcpcb.3dshapes/CRYSTAL-SMD_L3.2-W1.5-1.wrl"
 			(offset
 				(xyz 0 0 0)
@@
 		)
 	)
-	(footprint "MountingHole:MountingHole_2.7mm_M2.5"
+	(footprint "project:MountingHole_2.7mm_M2.5"
 		(locked yes)
 		(layer "F.Cu")
@@
 		)
 		(embedded_fonts no)
-		(model "${KIPRJMOD}/jlcpcb-lib/jlcpcb.3dshapes/R0603.wrl"
+		(model "${KIPRJMOD}/lib/jlcpcb/jlcpcb.3dshapes/R0603.wrl"
 			(offset
 				(xyz 0 0 0)
@@
 		)
 		(embedded_fonts no)
-		(model "${KIPRJMOD}/jlcpcb-lib/jlcpcb.3dshapes/R0603.wrl"
+		(model "${KIPRJMOD}/lib/jlcpcb/jlcpcb.3dshapes/R0603.wrl"
 			(offset
 				(xyz 0 0 0)
@@
 		)
 		(embedded_fonts no)
-		(model "${KIPRJMOD}/jlcpcb-lib/jlcpcb.3dshapes/R0603.wrl"
+		(model "${KIPRJMOD}/lib/jlcpcb/jlcpcb.3dshapes/R0603.wrl"
 			(offset
 				(xyz 0 0 0)
@@
 		)
 		(embedded_fonts no)
-		(model "${KIPRJMOD}/jlcpcb-lib/jlcpcb.3dshapes/C0603_L1.6-W0.8-H0.8.wrl"
+		(model "${KIPRJMOD}/lib/jlcpcb/jlcpcb.3dshapes/C0603_L1.6-W0.8-H0.8.wrl"
 			(offset
 				(xyz 0 0 0)
@@
 		)
 		(embedded_fonts no)
-		(model "${KIPRJMOD}/jlcpcb-lib/jlcpcb.3dshapes/R0603.wrl"
+		(model "${KIPRJMOD}/lib/jlcpcb/jlcpcb.3dshapes/R0603.wrl"
 			(offset
 				(xyz 0 0 0)
@@
 		)
 		(embedded_fonts no)
-		(model "${KIPRJMOD}/jlcpcb-lib/jlcpcb.3dshapes/R0603.wrl"
+		(model "${KIPRJMOD}/lib/jlcpcb/jlcpcb.3dshapes/R0603.wrl"
 			(offset
 				(xyz 0 0 0)
@@
 		)
 	)
-	(footprint "Connector_PinSocket_2.54mm:PinSocket_2x20_P2.54mm_Vertical"
+	(footprint "project:PinSocket_2x20_P2.54mm_Vertical"
 		(layer "B.Cu")
 		(at 108.37 48.77 -90)
@@
 		)
 		(embedded_fonts no)
-		(model "${KICAD10_3DMODEL_DIR}/Connector_PinSocket_2.54mm.3dshapes/PinSocket_2x20_P2.54mm_Vertical.step"
+		(model "${KIPRJMOD}/lib/project/project.3dshapes/PinSocket_2x20_P2.54mm_Vertical.step"
 			(offset
 				(xyz 0 0 0)
